File: PCB/Rev_0/BANDIT_Rev_0_0/BANDIT_Rev_0_0.kicad_sch (KiCad schematic)
At the start: 1 part, among them U1 RP2040

Commit message: Josh was here
Other:
- note added: "josh was here"
Changed lines of the file:
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@@
     (company "BODE Bandits: Team 9")
+  )
+  (text "josh was here\n" (at 161.29 101.6 0)
+    (effects (font (size 1.27 1.27)) (justify left bottom))
   )
   (text "BANDIT: Frequency Response Analyzer" (at 132.08 22.86 0)
