File: PCB/Dev_Platform/Bandit_Dev_Platform/Bandit_Dev_Platform.kicad_sch (KiCad schematic)
At the start: 112 parts, among them J1 Conn_01x03_Pin, J10 Conn_01x05_Pin, J11 Conn_01x05_Pin, J2 SMA, J3 Conn_01x05_Pin, J4 Conn_01x05_Pin, J5 BNC, J6 BNC, J7 SMA, J8 Conn_01x05_Pin, J9 Conn_01x06_Pin, P1 USB_C_Plug_USB2.0, SW1 SW_SPST, U1 AD7253, U1 OPA1664, U2 RP2040, U4 NCP164ASNADJT1G, U5 W25Q32JVSS, U6 MCP6486UT-E/OT, U7 MCP6S92-E/SN, Y1 12MHz

Commit message: started dev platform PCB
Parts:
- C1, C10, C11, C12, C13, C14, C15, C2, C23, C24, C26, C27, C28, C29, C3, C30, C31, C32, C33, C34, C35, C36, C37, C4, C5, C6, C7, C8, C9: footprint (none) -> Capacitor_SMD:C_0603_1608Metric
- C21, C22, C25: footprint (none) -> Capacitor_SMD:C_0805_2012Metric
- D1: footprint (none) -> LED_SMD:LED_0805_2012Metric
- D2: footprint (none) -> LED_SMD:LED_Cree-PLCC4_2x2mm_CW
- J1: footprint (none) -> Connector_PinHeader_2.54mm:PinHeader_1x03_P2.54mm_Vertical
- J10, J11, J3, J4, J8, J9: footprint (none) -> Connector_PinHeader_2.54mm:PinHeader_1x05_P2.54mm_Vertical
- JP1, JP2, JP3: footprint (none) -> Jumper:SolderJumper-2_P1.3mm_Open_TrianglePad1.0x1.5mm
- P1: footprint (none) -> Connector_USB:USB_C_Receptacle_GCT_USB4105-xx-A_16P_TopMnt_Horizontal
- R1, R10, R11, R12, R13, R2, R21, R22, R23, R24, R25, R26, R27, R3, R4, R5, R6, R7, R8, R9: footprint (none) -> Resistor_SMD:R_0603_1608Metric
- SW1: footprint (none) -> Button_Switch_THT:SW_PUSH_6mm
- U1: footprint (none) -> Package_SO:SOIC-14_3.9x8.7mm_P1.27mm
- U3: value ~ -> AP2210N-4.0TRG1; footprint (none) -> Package_TO_SOT_SMD:SOT-23-3
- Y1: footprint (none) -> Crystal:Crystal_SMD_EuroQuartz_MJ-4Pin_5.0x3.2mm
Connections:
- net FLASH_SCK: no longer U2.56 (QSPI_SS)
- net ~{FLASH_CSN}: now also U2.56 (QSPI_SS)
Other:
- moved on the sheet: C1, C12, C13, C14, C15, C2, C25, C3, C30, C31, C32, C4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
