File: PCB/Dev_Platform/Bandit_Dev_Platform/Bandit_Dev_Platform.kicad_sch (KiCad schematic)
At the start: 115 parts, among them J1 Conn_01x03_Pin, J10 Conn_01x05_Pin, J11 Conn_01x05_Pin, J2 SMA, J3 Conn_01x05_Pin, J4 Conn_01x05_Pin, J5 BNC, J6 BNC, J7 SMA, J8 Conn_01x05_Pin, J9 Conn_01x06_Pin, P1 USB_C_Plug_USB2.0, SW1 SW_SPST, U1 AD7253, U1 OPA1664, U2 RP2040, U3 AP2210N-4.0TRG1, U4 NCP164ASNADJT1G, U5 W25Q32JVSS, U6 MCP6486UT-E/OT, U7 MCP6S92-E/SN, X1 SG-210STF, Y1 12MHz

Commit message: Started 0402 transition, PN conversions for fabrication
Parts:
- C10, C7: value 15p COG -> 33p C0G
- U5: value W25Q32JVSS -> W25Q16JVUXIQ_TR; footprint Package_SO:SOIC-8_5.23x5.23mm_P1.27mm -> ICDB_Curly:IC_W25Q16JVUXIQ_TR
- Y1: value 12MHz -> 12.000 MHz, C9002; footprint Crystal:Crystal_SMD_EuroQuartz_MJ-4Pin_5.0x3.2mm -> Crystal:Crystal_SMD_3225-4Pin_3.2x2.5mm
Other:
- note added: "100n 0402: C307331 2u2 0402: C12530 10n 0402: C15195 1u 0402: C52923 10u 0402: C15525 1kR 0402: C11702"
- note added: "15p 0402: C1548 47p 0402: C1567 for 68: can do 2x C1562 33p 0402 in parallel 100p 0402: C1546"
- note added: "DO NOT INCLUDE!!"
- note added: "Note: Basic part at JLC so cheap, tested"
- note added: "Note: Footprint in ICDB Curly library, not dfl kicad"
- note added: "XTAL: C9002 Load Capacitors: C1562"
- note added: "for 16n Can either: 22n C1532 10n C15195 or maybe some dumb series thing"
Changed lines of the file:
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@@
     (stroke (width 0) (type default))
   )
+  (text "Note: Footprint in ICDB Curly library, not dfl kicad"
+    (at 40.64 156.21 0)
+    (effects (font (size 1.27 1.27)) (justify left bottom))
+  )
   (text "PGA: SPI1" (at 116.84 236.22 0)
     (effects (font (size 1.27 1.27)) (justify left bottom))
@@
     (effects (font (size 4 4) bold) (justify left bottom))
   )
+  (text "for 16n Can either:\n22n C1532\n10n C15195\nor maybe some dumb series thing"
+    (at 245.11 309.88 0)
+    (effects (font (size 1.27 1.27)) (justify left bottom))
+  )
   (text "ADC: SPI0 Single SDO or PIO for dual SDO" (at 116.84 219.71 0)
     (effects (font (size 1.27 1.27)) (justify left bottom))
@@
     (effects (font (size 1.27 1.27)) (justify left bottom))
   )
+  (text "DO NOT INCLUDE!!" (at 203.2 132.08 0)
+    (effects (font (size 1.27 1.27)) (justify left bottom))
+  )
   (text "FOR CLIPPY OPTION" (at 203.2 367.03 0)
     (effects (font (size 3 3) (thickness 0.6) bold) (justify left bottom))
   )
+  (text "Note: Basic part at JLC so cheap, tested" (at 72.39 344.17 0)
+    (effects (font (size 1.27 1.27)) (justify left bottom))
+  )
   (text "Could also... like be 10" (at 435.61 57.15 0)
     (effects (font (size 1.27 1.27)) (justify left bottom))
@@
     (effects (font (size 1.27 1.27)) (justify left bottom))
   )
+  (text "100n 0402: C307331\n2u2 0402: C12530\n10n 0402: C15195\n\n1u 0402: C52923\n10u 0402: C15525\n\n1kR 0402: C11702"
+    (at 162.56 186.69 0)
+    (effects (font (size 1.27 1.27)) (justify left bottom))
+  )
   (text "BANDIT Development Platform" (at 13.97 21.59 0)
     (effects (font (size 5 5) (thickness 1) bold) (justify left bottom))
@@
     (effects (font (size 4 4) bold) (justify left bottom))
   )
+  (text "XTAL: C9002\nLoad Capacitors: C1562" (at 72.39 349.25 0)
+    (effects (font (size 1.27 1.27)) (justify left bottom))
+  )
+  (text "15p 0402: C1548\n47p 0402: C1567\nfor 68: can do\n	2x C1562 33p 0402 in parallel\n\n100p 0402: C1546"
+    (at 353.06 209.55 0)
+    (effects (font (size 1.27 1.27)) (justify left bottom))
+  )
   (text "VEN_IH = 0.7V\nVEN_IL = 0.2V" (at 168.91 74.93 0)
     (effects (font (size 1.27 1.27)) (justify left bottom))
@@
       (effects (font (size 1.27 1.27)) (justify left))
     )
-    (property "Value" "15p COG" (at 55.88 342.8937 0)
+    (property "Value" "33p C0G" (at 55.88 342.8937 0)
       (effects (font (size 1.27 1.27)) (justify left))
     )
@@
       (effects (font (size 1.27 1.27)) (justify left))
     )
-    (property "Value" "W25Q32JVSS" (at 27.94 143.51 0)
+    (property "Value" "W25Q16JVUXIQ_TR" (at 27.94 143.51 0)
       (effects (font (size 1.27 1.27)) (justify left))
     )
-    (property "Footprint" "Package_SO:SOIC-8_5.23x5.23mm_P1.27mm" (at 36.83 142.24 0)
+    (property "Footprint" "ICDB_Curly:IC_W25Q16JVUXIQ_TR" (at 36.83 142.24 0)
       (effects (font (size 1.27 1.27)) hide)
     )
@@
       (effects (font (size 1.27 1.27)))
     )
-    (property "Value" "12MHz" (at 74.93 340.36 90)
+    (property "Value" "	12.000 MHz, C9002 " (at 74.93 340.36 90)
       (effects (font (size 1.27 1.27)))
     )
-    (property "Footprint" "Crystal:Crystal_SMD_EuroQuartz_MJ-4Pin_5.0x3.2mm" (at 53.34 335.28 0)
+    (property "Footprint" "Crystal:Crystal_SMD_3225-4Pin_3.2x2.5mm" (at 53.34 335.28 0)
       (effects (font (size 1.27 1.27)) hide)
     )
@@
       (effects (font (size 1.27 1.27)) (justify left))
     )
-    (property "Value" "15p COG" (at 55.88 323.8437 0)
+    (property "Value" "33p C0G" (at 55.88 323.8437 0)
       (effects (font (size 1.27 1.27)) (justify left))
     )

Commit message: Pcb kinda worked on
Parts:
- removed R13: 200R, Resistor_SMD:R_0603_1608Metric, symbol Device:R_Small_US
- added C2 (x2): 330p C0G, Capacitor_SMD:C_0402_1005Metric, symbol Device:C_Small
- added C4 (x2): 150p C0G, Capacitor_SMD:C_0402_1005Metric, symbol Device:C_Small
- added C5 (x2), C9 (x2): 68p C0G, Capacitor_SMD:C_0402_1005Metric, symbol Device:C_Small
- added C61, C62, C64, C65, C67: 100n, Capacitor_SMD:C_0402_1005Metric, symbol Device:C_Small
- added C63, C66: 2u2, Capacitor_SMD:C_0402_1005Metric, symbol Device:C_Small
- added C68: 10u, Capacitor_SMD:C_0402_1005Metric, symbol Device:C_Small
- added C69, C70, C71: 10u 0805, Capacitor_SMD:C_0805_2012Metric, symbol Device:C_Polarized_Small
- added FB1: FerriteBead_Small, Inductor_SMD:L_0603_1608Metric, symbol Device:FerriteBead_Small
- added R14: 1k, Resistor_SMD:R_0402_1005Metric, symbol Device:R_Small_US
- added U8: MIC5504-3.3YM5, Package_TO_SOT_SMD:SOT-23-5, symbol Regulator_Linear:MIC5504-3.3YM5
- C1, C10, C11, C12, C13, C14, C15, C17, C18, C2, C23, C24, C26, C27, C28, C29, C3, C30, C31, C32, C33, C34, C35, C36, C37, C4, C5, C6, C7, C8, C9: footprint Capacitor_SMD:C_0603_1608Metric -> Capacitor_SMD:C_0402_1005Metric
- C21, C22: footprint Capacitor_SMD:C_0805_2012Metric -> Capacitor_SMD:C_0402_1005Metric
- C25: value C_Polarized_Small -> 10u 0805
- J2: footprint (none) -> Capacitor_SMD:C_0402_1005Metric
- R1, R2, R3, R6: value 200R -> 330R; footprint Resistor_SMD:R_0603_1608Metric -> Resistor_SMD:R_0402_1005Metric
- R12, R21, R22, R23, R24, R27, R4, R5: footprint Resistor_SMD:R_0603_1608Metric -> Resistor_SMD:R_0402_1005Metric
- R25, R26: value 50k -> 51k; footprint Resistor_SMD:R_0603_1608Metric -> Resistor_SMD:R_0402_1005Metric
- R7: footprint Resistor_SMD:R_0603_1608Metric -> Resistor_SMD:R_0805_2012Metric
Connections:
- net +1V1: now also C62.1, C63.1, C64.1
- net +3V3: now also C61.1, C65.1, C66.1, C67.1, C68.1, C69.1, FB1.2, U8.5 (VOUT)
- net GND: now also C61.2, C62.2, C63.2, C64.2, C65.2, C66.2, C67.2, C68.2, C69.2, C70.2, U8.2 (GND); no longer C8.2, C9.2, R9.1
- net GNDA: now also C8.2, C9.2, R9.1, C5.1, C5.1, C71.2, C9.1, C9.1
- net SE_SIG_A: now also C2.1
- net SE_SIG_B: now also C2.1
- net VBUS: now also C70.1, U8.1 (VIN)
- net VDDA: now also C71.1
- net XOUT: now also R14.2; no longer U2.21 (XOUT)
- net at C4.2, R3.1, R4.2: now also C4.2 (x2)
- net at C4.1, R2.1, U1.1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: now also C4.1
- net at C2.2, R1.1, R2.2: now also C2.2 (x2)
- net at C5.2, R5.2, U1.3 (+): now also C5.2
- net at C11.1, U2.43 (ADC_AVDD): now also FB1.1
- net at C4.1, R2.1, U1.6 (-)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: now also C4.1
- net at C5.2, R5.2, U1.5 (+): now also C5.2
- net at C9.2, R7.2, U1.12 (+): now also C9.2
- net at C9.2, R7.2, U1.10 (+): now also C9.2
- new net: R14.1, U2.21 (XOUT)
Other:
- note added: "100p + 47p = 147p"
- note added: "10R 0402: C25077"
- note added: "10u 0805: C440198"
- note added: "150k 0402: C22807 51k 0402: C25794 49.9k 0603: C23184"
- note added: "15p 0402: C1548 47p 0402: C1567 for 68: can do 2x C1562 33p 0402 in parallel 100p 0402: C1546 6k2 0603: C4260 15k 0402: C25756"
- note added: "220p + 100p = 320p"
- note added: "330R 0402: C25104"
- note added: "51k 0402: C25794"
- note added: "Vref_adj = 1.10V Vout = Vfix * (1 + R1 / R2) Note: R1 and R2 should both be < 500k 4.096 = 1.1 * (1 + R1 / 50e3) Pick R2 = 50k R1 = 149,800 ~= 150k Alt: fix R1 = 150k 4.096 = 1.1 * (1 + 150k / R2) R2 = 55073 = 55k"
- note added: "for 16n Can either: 22n C1532 10n C15195 or maybe some dumb series thing 22R 0402: C25092"
- note removed: "15p 0402: C1548 47p 0402: C1567 for 68: can do 2x C1562 33p 0402 in parallel 100p 0402: C1546"
- note removed: "Vref_adj = 1.10V Vout = Vfix * (1 + R1 / R2) Note: R1 and R2 should both be < 500k 4.096 = 1.1 * (1 + R1 / 50e3) Pick R2 = 50k R1 = 149,800 ~= 150k"
- note removed: "for 16n Can either: 22n C1532 10n C15195 or maybe some dumb series thing"
