File: PCB/Dev_Platform/Bandit_Dev_Platform/Bandit_Dev_Platform.kicad_pcb (KiCad board)
At the start: 4 copper layers, 63.5 x 31.8 mm, 113 parts, among them J1 Conn_01x03_Pin, J10 Conn_01x05_Pin, J11 Conn_01x05_Pin, J3 Conn_01x05_Pin, J4 Conn_01x05_Pin, J5 BNC, J6 BNC, J8 Conn_01x05_Pin, J9 Conn_01x06_Pin, P1 USB_C_Plug_USB2.0, SW1 SW_SPST, U1 AD7253, U10 OPA1664, U2 RP2040, U3 AP2210N-4.0TRG1, U4 NCP164ASNADJT1G, U5 W25Q32JVSS, U6 MCP6486UT-E/OT, U7 MCP6S92-E/SN, U9 OPA1664, X1 SG-210STF, Y1 12MHz

Commit message: PCB Updates
Parts:
- moved U6 110.8 mm to (40.3, 23.9), turned to 90 degrees
- moved R27 90.8 mm to (37.5, 25.9), turned to -90 degrees
- moved C21 86.5 mm to (50.9, 41.0), turned to 90 degrees
- moved U7 79.6 mm to (67.0, 34.0), turned to 180 degrees
- moved R22 69.9 mm to (49.8, 33.1), turned to 180 degrees
- moved R21 68.1 mm to (49.8, 34.6), turned to 180 degrees
- moved R24 64.7 mm to (55.9, 37.7), turned to 180 degrees
- moved R23 62.7 mm to (55.9, 39.4), turned to 180 degrees
- moved C23 60.6 mm to (47.5, 33.8), turned to -90 degrees
- moved C24 54.1 mm to (53.6, 39.1), turned to 90 degrees
- moved U1 8.98 mm to (45.2, 42.9)
- moved C55 7.26 mm to (62.0, 27.5)
- moved R39 7.26 mm to (62.0, 28.9)
- moved C41 7.26 mm to (56.6, 34.0)
- moved C51 7.26 mm to (53.6, 34.0)
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
Commit message: Pcb kinda worked on
Parts:
- added C16: 68p C0G, Capacitor_SMD:C_0402_1005Metric, F.Cu at (70.9, 78.5)
- added C19: 68p C0G, Capacitor_SMD:C_0402_1005Metric, F.Cu at (70.9, 84.4)
- added C20: 68p C0G, Capacitor_SMD:C_0402_1005Metric, F.Cu at (70.9, 86.3)
- added C38: 68p C0G, Capacitor_SMD:C_0402_1005Metric, F.Cu at (76.6, 76.5)
- added C39: 330p C0G, Capacitor_SMD:C_0402_1005Metric, F.Cu at (76.6, 78.5)
- added C40: 330p C0G, Capacitor_SMD:C_0402_1005Metric, F.Cu at (76.6, 80.4)
- added C59: 150p C0G, Capacitor_SMD:C_0402_1005Metric, F.Cu at (82.3, 74.5)
- added C60: 150p C0G, Capacitor_SMD:C_0402_1005Metric, F.Cu at (82.3, 76.5)
- added C61: 100n, Capacitor_SMD:C_0402_1005Metric, F.Cu at (34.6, 33.6)
- added C62: 100n, Capacitor_SMD:C_0402_1005Metric, F.Cu at (33.0, 34.8)
- added C63: 2u2, Capacitor_SMD:C_0402_1005Metric, F.Cu at (33.0, 33.8)
- added C64: 100n, Capacitor_SMD:C_0402_1005Metric, F.Cu at (44.1, 35.4)
- added C65: 100n, Capacitor_SMD:C_0402_1005Metric, F.Cu at (45.1, 35.1)
- added C66: 2u2, Capacitor_SMD:C_0402_1005Metric, F.Cu at (46.1, 35.1)
- added C67: 100n, Capacitor_SMD:C_0402_1005Metric, F.Cu at (30.4, 27.0)
- added C68: 10u, Capacitor_SMD:C_0402_1005Metric, F.Cu at (31.4, 27.0)
- added C69: 10u 0805, Capacitor_SMD:C_0805_2012Metric, F.Cu at (28.1, 24.6)
- added C70: 10u 0805, Capacitor_SMD:C_0805_2012Metric, F.Cu at (45.0, 23.2)
- added C71: 10u 0805, Capacitor_SMD:C_0805_2012Metric, F.Cu at (55.1, 23.2)
- added FB1: FerriteBead_Small, Inductor_SMD:L_0603_1608Metric, F.Cu at (34.5, 30.8)
- added J2: SMA, Capacitor_SMD:C_0402_1005Metric, F.Cu at (82.3, 78.5)
- added R14: 1k, Resistor_SMD:R_0402_1005Metric, F.Cu at (46.4, 36.6)
- added U8: MIC5504-3.3YM5, Package_TO_SOT_SMD:SOT-23-5, F.Cu at (27.7, 27.4)
- C1, C11, C12, C13, C14, C15, C17, C18, C2, C26, C27, C28, C29, C3, C30, C31, C32, C33, C34, C35, C36, C37, C4, C41, C42, C43, C44, C45, C46, C47, C48, C49, C5, C50, C51, C52, C53, C54, C55, C56, C57, C58, C6, C8, C9: footprint Capacitor_SMD:C_0603_1608Metric -> Capacitor_SMD:C_0402_1005Metric
- C10, C7: value 15p COG -> 33p C0G; footprint Capacitor_SMD:C_0603_1608Metric -> Capacitor_SMD:C_0402_1005Metric
- C21, C22: footprint Capacitor_SMD:C_0805_2012Metric -> Capacitor_SMD:C_0402_1005Metric
- C23, C24: value 36n C0G -> 16n C0G; footprint Capacitor_SMD:C_0603_1608Metric -> Capacitor_SMD:C_0402_1005Metric
- C25: value C_Polarized_Small -> 10u 0805
- R1, R2, R3, R6: value 200R -> 330R; footprint Resistor_SMD:R_0603_1608Metric -> Resistor_SMD:R_0402_1005Metric
- R12, R13, R27, R4, R5: footprint Resistor_SMD:R_0603_1608Metric -> Resistor_SMD:R_0402_1005Metric
- R21, R22, R23, R24: value 10R -> 20R; footprint Resistor_SMD:R_0603_1608Metric -> Resistor_SMD:R_0402_1005Metric
- R25, R26: value 50k -> 51k; footprint Resistor_SMD:R_0603_1608Metric -> Resistor_SMD:R_0402_1005Metric
- R7: footprint Resistor_SMD:R_0603_1608Metric -> Resistor_SMD:R_0805_2012Metric
- U5: value W25Q32JVSS -> W25Q16JVUXIQ_TR; footprint Package_SO:SOIC-8_5.23x5.23mm_P1.27mm -> ICDB_Curly:IC_W25Q16JVUXIQ_TR
- Y1: value 12MHz -> 12.000 MHz, C9002; footprint Crystal:Crystal_SMD_EuroQuartz_MJ-4Pin_5.0x3.2mm -> Crystal:Crystal_SMD_3225-4Pin_3.2x2.5mm
- moved SW1 115.9 mm to (23.1, 44.8)
- moved JP2 105.0 mm to (45.5, 26.2), turned to 180 degrees
- moved U4 101.3 mm to (50.1, 23.2)
- moved R10 92.7 mm to (29.7, 33.1), turned to 90 degrees
- moved J9 91.4 mm to (41.8, 24.2), turned to -90 degrees
- moved R11 91.1 mm to (29.7, 38.6), turned to -90 degrees
- moved Y1 90.8 mm to (47.6, 38.8), turned to 180 degrees
- moved C22 89.7 mm to (47.3, 45.8), turned to 90 degrees
- moved C6 81.5 mm to (23.8, 25.4), turned to 180 degrees
- moved C5 80.7 mm to (23.8, 24.4), turned to 180 degrees
- moved C4 78.3 mm to (23.8, 26.4), turned to 180 degrees
- moved R9 77.8 mm to (51.0, 27.4), turned to 180 degrees
- moved R8 77.0 mm to (51.3, 25.8)
- moved R7 77.0 mm to (48.3, 26.7), turned to 90 degrees
- moved C11 76.3 mm to (35.0, 32.1), turned to 180 degrees
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Connections:
- C8 pad 2: GND -> GNDA
- C9 pad 2: GND -> GNDA
- R9 pad 1: GND -> GNDA
- U2 pad 21: /XOUT -> Net-(U2-XOUT)
Routing:
- net VBUS: track 0.00 -> 46.0 mm
- net /WGN_OUT: track 0.00 -> 33.1 mm
- net +1V1: track 0.00 -> 26.6 mm
- net GND: track 0.00 -> 21.2 mm, vias 0 -> 50
- net +3V3: track 0.00 -> 18.3 mm, vias 0 -> 15
- net /FLASH_IO3: track 22.5 -> 6.79 mm
- net /FLASH_SCK: track 19.9 -> 5.75 mm
- net Net-(C54-Pad2): track 12.9 -> 0.00 mm
- net /FLASH_IO0: track 17.1 -> 4.54 mm
- net Net-(C45-Pad2): track 12.2 -> 0.00 mm
- net Net-(J9-Pin_5): track 0.00 -> 11.7 mm
- net Net-(U10B-+): track 11.3 -> 0.00 mm
- net Net-(J9-Pin_4): track 0.00 -> 10.8 mm
- net Net-(J9-Pin_3): track 0.00 -> 9.92 mm
- net Net-(J9-Pin_2): track 0.00 -> 9.73 mm
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- added copper zone on F.Cu, net +3V3
- added copper zone on In1.Cu, net +3V3
- added copper zone on F.Cu, net GND
- added copper zone on In2.Cu, net GND
- added copper zone on F.Cu, net GNDA
- added copper zone on In2.Cu, net GNDA
- added copper zone on In1.Cu, net VDDA
- removed copper zone on F.Cu, net /SE_SIG_A
- removed copper zone on F.Cu, net /SE_SIG_B
- removed copper zone on In1.Cu, net GND
- removed copper zone on In1.Cu, net GNDA
- removed copper zone on F.Cu, net Net-(U10A--)
- removed copper zone on F.Cu, net Net-(U10B--)
- removed copper zone on F.Cu, net Net-(U10D--)
- removed copper zone on F.Cu, net Net-(U9A--)
- removed copper zone on F.Cu, net Net-(U9B--)
- removed copper zone on F.Cu, net Net-(U9C--)
