File: PCB/Dev_Platform/Bandit_Dev_Platform/Bandit_Dev_Platform.kicad_pcb (KiCad board)
At the start: 4 copper layers, 63.5 x 31.8 mm, 135 parts, among them J1 Conn_01x03_Pin, J10 Conn_01x05_Pin, J11 Conn_01x05_Pin, J2 SMA, J3 Conn_01x05_Pin, J4 Conn_01x05_Pin, J5 BNC, J6 BNC, J8 Conn_01x05_Pin, J9 Conn_01x06_Pin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

Commit message: Done?
Parts:
- removed C12, C15, C17: 100n, Capacitor_SMD:C_0402_1005Metric
- removed C18: 10n, Capacitor_SMD:C_0402_1005Metric
- removed J1: Conn_01x03_Pin, Connector_PinHeader_2.54mm:PinHeader_1x03_P2.54mm_Vertical
- removed J10, J11, J3, J4, J8: Conn_01x05_Pin, Connector_PinHeader_2.54mm:PinHeader_1x05_P2.54mm_Vertical
- removed J2: SMA, Capacitor_SMD:C_0402_1005Metric
- removed J9: Conn_01x06_Pin, Connector_PinHeader_2.54mm:PinHeader_1x05_P2.54mm_Vertical
- removed JP1, JP3: SolderJumper_2_Open, Jumper:SolderJumper-2_P1.3mm_Open_TrianglePad1.0x1.5mm
- removed U3: AP2210N-4.0TRG1, Package_TO_SOT_SMD:SOT-23-3
- removed X1: SG-210STF, Oscillator:Oscillator_SMD_SeikoEpson_SG210-4Pin_2.5x2.0mm
- added C72: 10u 0805, Capacitor_SMD:C_0805_2012Metric, F.Cu at (76.0, 33.8)
- added C73: 10u 0805, Capacitor_SMD:C_0805_2012Metric, F.Cu at (68.2, 26.4)
- added C74: 100n, Capacitor_SMD:C_0402_1005Metric, F.Cu at (40.2, 28.0)
- added G***: LOGO, BANDIT_PCB_Lib:Logo_30mm, B.Cu at (40.4, 35.8)
- added J12: Conn_01x02_Pin, Connector_PinSocket_2.54mm:PinSocket_1x02_P2.54mm_Vertical, F.Cu at (68.4, 22.7)
- added R13: 51k, Resistor_SMD:R_0402_1005Metric, F.Cu at (78.7, 34.2)
- added R15: 51k, Resistor_SMD:R_0402_1005Metric, F.Cu at (77.6, 34.2)
- moved R12 79.0 mm to (32.4, 42.1), turned to -135 degrees
- moved C35 67.8 mm to (37.5, 27.7), turned to 90 degrees
- moved C31 57.6 mm to (66.5, 37.1), turned to 90 degrees
- moved C30 56.2 mm to (65.5, 36.9), turned to 90 degrees
- moved SW1 0.70 mm to (23.1, 44.1)
- moved JP2 0.65 mm to (42.9, 26.6), turned to -90 degrees
- moved C25 0.47 mm to (76.0, 37.9)
- moved R25 0.47 mm to (78.7, 37.5)
- moved R26 0.47 mm to (77.6, 37.5)
- moved C20 0.44 mm to (61.6, 36.0)
- moved C55 0.44 mm to (61.9, 26.5)
- moved C56 0.44 mm to (64.4, 29.4)
- moved C59 0.44 mm to (55.1, 26.5)
- moved R39 0.44 mm to (64.4, 27.6)
- moved R40 0.44 mm to (64.7, 32.1)
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Connections:
- J6 pad 1: /WGN_OUT -> /WGN_OUT_PORT
- R41 pad 1: /WGN_OUT -> /WGN_PGA_IN
- U7 pad 3: /WGN_OUT -> /WGN_PGA_IN
Routing:
- net /~{PGA_CS}: track 1.22 -> 42.8 mm, vias 1 -> 2
- net /PGA_SCK: track 1.23 -> 42.6 mm, vias 1 -> 2
- net /PGA_SI: track 1.14 -> 41.9 mm, vias 1 -> 2
- net /WGN_OUT: track 46.5 -> 23.0 mm
- net /USER_LED: track 0.00 -> 20.7 mm, vias 0 -> 2
- net /WGN_PGA_IN: track 0.00 -> 17.6 mm
- net /WGN_OUT_PORT: track 0.00 -> 17.3 mm
- net /LED_R: track 0.00 -> 15.3 mm, vias 0 -> 2
- net /LED_G: track 0.00 -> 13.5 mm, vias 0 -> 2
- net /LED_B: track 0.00 -> 13.3 mm, vias 0 -> 2
- net GND: track 37.1 -> 45.6 mm, vias 86 -> 98
- net +3V3: track 19.3 -> 22.6 mm, vias 17 -> 18
- net /~{FLASH_CSN}: track 6.95 -> 10.1 mm
- net Net-(SW1-A): track 0.00 -> 3.17 mm
- net VDDA: track 22.2 -> 25.2 mm, vias 11 -> 15
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Other:
- board text added: "BANDIT"
- board text added: "BANDIT V1.0"
- board text added: "C. Abella A. Bergado J. Cole J. De Vico L. Reyes"
- board text added: "HELLO"

Commit message: More done
Parts:
- moved C28 0.12 mm to (36.8, 38.6)
- moved C29 0.12 mm to (36.8, 39.6)
Connections:
- U5 pad 9: (no net) -> GND
Routing:
- net +3V3: track 22.6 -> 25.7 mm, vias 18 -> 19
- net /ADC_SCK: track 1.51 -> 4.55 mm, vias 0 -> 2
- net /ADC_CSN: track 1.43 -> 3.85 mm, vias 1 -> 2
- net +1V1: track 24.6 -> 23.6 mm
